File: ergogen/output/pcbs/left.kicad_pcb (KiCad board)
At the start: 2 copper layers, 140.6 x 129.2 mm, 24 parts

Commit message: getting closer to a design I like
Parts:
- removed the REF** at (169.6, 109.4)
- removed the REF** at (193.7, 115.9)
- removed the REF** at (212.6, 132.2)
- added REF**: ks27, gateron-ks27-hotswap-reversible, F.Cu at (157.6, 110.4)
- added REF**: ks27, gateron-ks27-hotswap-reversible, F.Cu at (180.7, 113.5)
- added REF**: ks27, gateron-ks27-hotswap-reversible, F.Cu at (202.6, 121.8)
- moved MCU1 79.5 mm to (96.2, 33.1), turned to 5 degrees
Other:
- board size 140.6 x 129.2 mm -> 131.3 x 118.5 mm
