File: pcb/left.kicad_sch (KiCad schematic)
At the start: 83 parts, among them SW1 Key Switch, SW10 Key Switch, SW11 Key Switch, SW12 Key Switch, SW13 Key Switch, SW14 Key Switch, SW15 Key Switch, SW16 Key Switch, SW17 Key Switch, SW18 Key Switch, SW19 Key Switch, SW2 Key Switch, SW20 Key Switch, SW21 Key Switch, SW22 Key Switch, SW23 Key Switch, SW24 Program Btn, SW3 Key Switch, SW4 Key Switch, SW5 Key Switch, SW6 Key Switch, SW7 Key Switch, SW8 Key Switch, SW9 Key Switch, Sw27 SW_Push, Sw28 SW_SPDT, U4 Shift Register, U5 SeeeduinoXIAO_BLE, U6 Level Shifter

Commit message: starting to work on the ergogen side again
Connections:
- net Row3: no longer U5.5 (PA8_A4_D4_SDA)
- net Row4: now also U5.5 (PA8_A4_D4_SDA)
Changed lines of the file:
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@@
 		)
 	)
-	(global_label "Row3"
+	(global_label "Row4"
 		(shape input)
 		(at 74.93 165.1 180)
