File: pcb/left.kicad_sch (KiCad schematic)
At the start: 84 parts, among them SW1 Key Switch, SW10 Key Switch, SW11 Key Switch, SW12 Key Switch, SW13 Key Switch, SW14 Key Switch, SW15 Key Switch, SW16 Key Switch, SW17 Key Switch, SW18 Key Switch, SW19 Key Switch, SW2 Key Switch, SW20 Key Switch, SW21 Key Switch, SW22 Key Switch, SW23 Key Switch, SW24 Program Btn, SW3 Key Switch, SW4 Key Switch, SW5 Key Switch, SW6 Key Switch, SW7 Key Switch, SW8 Key Switch, SW9 Key Switch, Sw27 SW_Push, Sw28 SW_SPDT, U1 SeeeduinoXIAO_BLE, U2 Shift Register, U3 Level Shifter

Commit message: sooo close
Connections:
- net Row0: now also D1.1 (K); no longer D24.1 (K)
- net Row1: now also D6.1 (K); no longer D1.1 (K)
- net Row2: now also D11.1 (K); no longer D6.1 (K)
- net Row3: now also D16.1 (K); no longer D11.1 (K)
- net Row4: now also D24.1 (K); no longer D16.1 (K)
Other:
- moved on the sheet: D1, D11, D16, D24, D6, SW1, SW11, SW16, SW24, SW6

Commit message: SOO CLOSE
Parts:
- removed C1: 1000 uF, symbol Device:C
- added LED28, LED30: SK6812MINI, LED_SMD:LED_SK6812MINI_PLCC4_3.5x3.5mm_P1.75mm, symbol LED:SK6812MINI
- renumbered D17 to D1, D14 to D10, D9 to D11, D4 to D12, D20 to D13, D15 to D14, D10 to D15, D5 to D16, D21 to D17, D22 to D18, D23 to D19, D12 to D2, D16 to D20, D11 to D21, D6 to D22, D1 to D23, D7 to D3, D2 to D4, D18 to D5, D13 to D6, D8 to D7, D3 to D8, D19 to D9, LED26 to LED25, LED27 to LED26, LED28 to LED27, LED25 to LED29, LED29 to LED31, SW16 to SW1, SW13 to SW10, SW8 to SW11, SW3 to SW12, SW19 to SW13, SW9 to SW15, SW4 to SW16, SW20 to SW17, SW15 to SW18, SW10 to SW19, SW11 to SW2, SW5 to SW20, SW6 to SW3, SW1 to SW4, SW17 to SW5, SW12 to SW6, SW2 to SW8, SW18 to SW9
Connections:
- net +5V: now also LED1.2 (VSS), LED10.2 (VSS), LED11.2 (VSS), LED12.2 (VSS), LED13.2 (VSS), LED14.2 (VSS), LED15.2 (VSS), LED16.2 (VSS), LED17.2 (VSS), LED18.2 (VSS), LED19.2 (VSS), LED2.2 (VSS), LED20.2 (VSS), LED21.2 (VSS), LED22.2 (VSS), LED23.2 (VSS), LED24.2 (VSS), LED25.2 (VSS), LED26.2 (VSS), LED27.2 (VSS), LED29.2 (VSS), LED3.2 (VSS), LED31.2 (VSS), LED4.2 (VSS), LED5.2 (VSS), LED6.2 (VSS), LED7.2 (VSS), LED8.2 (VSS), LED9.2 (VSS), LED28.2 (VSS), LED30.2 (VSS); no longer LED1.4 (VDD), LED10.4 (VDD), LED11.4 (VDD), LED12.4 (VDD), LED13.4 (VDD), LED14.4 (VDD), LED15.4 (VDD), LED16.4 (VDD), LED17.4 (VDD), LED18.4 (VDD), LED19.4 (VDD), LED2.4 (VDD), LED20.4 (VDD), LED21.4 (VDD), LED22.4 (VDD), LED23.4 (VDD), LED24.4 (VDD), LED25.4 (VDD), LED26.4 (VDD), LED27.4 (VDD), LED29.4 (VDD), LED3.4 (VDD), LED31.4 (VDD), LED4.4 (VDD), LED5.4 (VDD), LED6.4 (VDD), LED7.4 (VDD), LED8.4 (VDD), LED9.4 (VDD)
- net +BATT: now also Sw28.1 (A); no longer BT2.1 (+)
- net Backlight LED: now also LED1.1 (DOUT), LED24.3 (DIN); no longer LED23.1 (DOUT), LED27.3 (DIN)
- net GND: now also BT2.2 (-), LED1.4 (VDD), LED10.4 (VDD), LED11.4 (VDD), LED12.4 (VDD), LED13.4 (VDD), LED14.4 (VDD), LED15.4 (VDD), LED16.4 (VDD), LED17.4 (VDD), LED18.4 (VDD), LED19.4 (VDD), LED2.4 (VDD), LED20.4 (VDD), LED21.4 (VDD), LED22.4 (VDD), LED23.4 (VDD), LED24.4 (VDD), LED25.4 (VDD), LED26.4 (VDD), LED27.4 (VDD), LED29.4 (VDD), LED3.4 (VDD), LED31.4 (VDD), LED4.4 (VDD), LED5.4 (VDD), LED6.4 (VDD), LED7.4 (VDD), LED8.4 (VDD), LED9.4 (VDD), LED28.4 (VDD), LED30.4 (VDD); no longer LED1.2 (VSS), LED10.2 (VSS), LED11.2 (VSS), LED12.2 (VSS), LED13.2 (VSS), LED14.2 (VSS), LED15.2 (VSS), LED16.2 (VSS), LED17.2 (VSS), LED18.2 (VSS), LED19.2 (VSS), LED2.2 (VSS), LED20.2 (VSS), LED21.2 (VSS), LED22.2 (VSS), LED23.2 (VSS), LED24.2 (VSS), LED25.2 (VSS), LED26.2 (VSS), LED27.2 (VSS), LED29.2 (VSS), LED3.2 (VSS), LED31.2 (VSS), LED4.2 (VSS), LED5.2 (VSS), LED6.2 (VSS), LED7.2 (VSS), LED8.2 (VSS), LED9.2 (VSS), Sw28.2 (B)
- net LED: now also LED23.3 (DIN); no longer LED1.3 (DIN)
- net at LED29.1 (DOUT): now also LED31.3 (DIN)
- net at LED29.3 (DIN): now also LED30.1 (DOUT); no longer LED31.1 (DOUT)
- net at LED20.1 (DOUT): now also LED15.3 (DIN); no longer LED23.3 (DIN)
- net at LED20.3 (DIN): now also LED19.1 (DOUT); no longer LED15.1 (DOUT)
- net at LED5.1 (DOUT): now also LED4.3 (DIN); no longer LED10.3 (DIN)
- net at LED5.3 (DIN): now also LED10.1 (DOUT); no longer LED4.1 (DOUT)
- net at LED22.1 (DOUT): now also LED21.3 (DIN); no longer LED19.3 (DIN)
- net at LED22.3 (DIN): now also LED23.1 (DOUT); no longer LED21.1 (DOUT)
- net at LED27.1 (DOUT): now also LED28.3 (DIN); no longer LED26.3 (DIN)
- net at LED9.1 (DOUT): now also LED10.3 (DIN); no longer LED4.3 (DIN)
- net at LED9.3 (DIN): now also LED8.1 (DOUT); no longer LED14.1 (DOUT)
- net at LED7.1 (DOUT): now also LED8.3 (DIN); no longer LED2.3 (DIN)
- net at LED7.3 (DIN): now also LED6.1 (DOUT); no longer LED12.1 (DOUT)
- net at LED25.1 (DOUT): now also LED26.3 (DIN); no longer LED24.3 (DIN)
- net at LED26.1 (DOUT): now also LED27.3 (DIN); no longer LED25.3 (DIN)
- net at LED14.3 (DIN): now also LED15.1 (DOUT); no longer LED19.1 (DOUT)
- net at LED12.3 (DIN): now also LED13.1 (DOUT); no longer LED17.1 (DOUT)
- net at LED18.1 (DOUT): now also LED19.3 (DIN); no longer LED21.3 (DIN)
- net at LED18.3 (DIN): now also LED17.1 (DOUT); no longer LED13.1 (DOUT)
- net at LED13.3 (DIN): now also LED14.1 (DOUT); no longer LED8.1 (DOUT)
- net at LED3.1 (DOUT): now also LED2.3 (DIN); no longer LED8.3 (DIN)
- net at LED11.1 (DOUT): now also LED6.3 (DIN); no longer LED16.3 (DIN)
- net at LED11.3 (DIN): now also LED12.1 (DOUT); no longer LED6.1 (DOUT)
- net at LED3.3 (DIN): now also LED4.1 (DOUT); no longer LED2.1 (DOUT)
- net at LED24.1 (DOUT): now also LED25.3 (DIN); no longer LED31.3 (DIN)
- new net: LED28.1 (DOUT), LED30.3 (DIN)
- new net: LED1.3 (DIN), LED2.1 (DOUT)
- new net: LED16.3 (DIN), LED21.1 (DOUT)
- new net: BT2.1 (+), Sw28.2 (B)
Other:
- moved on the sheet: BT2, LED1, LED10, LED11, LED12, LED13, LED14, LED15, LED16, LED17, LED18, LED19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

Commit message: trying to make mcu_cover
Parts:
- renumbered BT2 to JST1, LED16 to LED1, LED13 to LED10, LED8 to LED11, LED3 to LED12, LED19 to LED13, LED9 to LED15, LED4 to LED16, LED20 to LED17, LED15 to LED18, LED10 to LED19, LED11 to LED2, LED5 to LED20, LED6 to LED3, LED1 to LED4, LED17 to LED5, LED12 to LED6, LED2 to LED8, LED18 to LED9, Sw27 to Sw25
Changed lines of the file:
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@@
 		(on_board yes)
 		(dnp no)
-		(property "Reference" "LED20"
+		(property "Reference" "LED17"
 			(at 257.556 92.456 0)
 			(effects
@@
 			(project "left"
 				(path "/354a5e63-d0f6-4612-b9d9-61a572cb8576"
-					(reference "LED20")
+					(reference "LED17")
 					(unit 1)
 				)
@@
 		(on_board yes)
 		(dnp no)
-		(property "Reference" "LED5"
-			(at 256.794 27.686 0)
+		(property "Reference" "LED20"
+			(at 257.302 27.686 0)
 			(effects
 				(font
@@
 			(project "left"
 				(path "/354a5e63-d0f6-4612-b9d9-61a572cb8576"
-					(reference "LED5")
+					(reference "LED20")
 					(unit 1)
 				)
@@
 		(on_board yes)
 		(dnp no)
-		(property "Reference" "LED9"
+		(property "Reference" "LED15"
 			(at 230.124 49.276 0)
 			(effects
@@
 			(project "left"
 				(path "/354a5e63-d0f6-4612-b9d9-61a572cb8576"
-					(reference "LED9")
+					(reference "LED15")
 					(unit 1)
 				)
@@
 		(on_board yes)
 		(dnp no)
-		(property "Reference" "LED4"
-			(at 230.124 27.686 0)
+		(property "Reference" "LED16"
+			(at 230.886 27.686 0)
 			(effects
 				(font
@@
 			(project "left"
 				(path "/354a5e63-d0f6-4612-b9d9-61a572cb8576"
-					(reference "LED4")
+					(reference "LED16")
 					(unit 1)
 				)
@@
 		(on_board yes)
 		(dnp no)
-		(property "Reference" "LED10"
+		(property "Reference" "LED19"
 			(at 257.556 49.276 0)
 			(effects
@@
 			(project "left"
 				(path "/354a5e63-d0f6-4612-b9d9-61a572cb8576"
-					(reference "LED10")
+					(reference "LED19")
 					(unit 1)
 				)
@@
 		(dnp no)
 		(fields_autoplaced yes)
-		(property "Reference" "Sw27"
+		(property "Reference" "Sw25"
 			(at 147.32 142.24 0)
 			(effects
@@
 			(project "left"
 				(path "/354a5e63-d0f6-4612-b9d9-61a572cb8576"
-					(reference "Sw27")
+					(reference "Sw25")
 					(unit 1)
 				)
@@
 		(on_board yes)
 		(dnp no)
-		(property "Reference" "LED19"
+		(property "Reference" "LED13"
 			(at 230.886 92.456 0)
 			(effects
@@
 			(project "left"
 				(path "/354a5e63-d0f6-4612-b9d9-61a572cb8576"
-					(reference "LED19")
+					(reference "LED13")
 					(unit 1)
 				)
@@
 		(on_board yes)
 		(dnp no)
-		(property "Reference" "LED12"
-			(at 177.546 70.866 0)
+		(property "Reference" "LED6"
+			(at 177.038 70.866 0)
 			(effects
 				(font
@@
 			(project "left"
 				(path "/354a5e63-d0f6-4612-b9d9-61a572cb8576"
-					(reference "LED12")
+					(reference "LED6")
 					(unit 1)
 				)
@@
 		(on_board yes)
 		(dnp no)
-		(property "Reference" "LED2"
+		(property "Reference" "LED8"
 			(at 176.784 27.7562 0)
 			(effects
@@
 			(project ""
 				(path "/354a5e63-d0f6-4612-b9d9-61a572cb8576"
-					(reference "LED2")
+					(reference "LED8")
 					(unit 1)
 				)
@@
 		(on_board yes)
 		(dnp no)
-		(property "Reference" "LED18"
+		(property "Reference" "LED9"
 			(at 204.216 92.456 0)
 			(effects
@@
 			(project "left"
 				(path "/354a5e63-d0f6-4612-b9d9-61a572cb8576"
-					(reference "LED18")
+					(reference "LED9")
 					(unit 1)
 				)
@@
 		(on_board yes)
 		(dnp no)
-		(property "Reference" "LED8"
-			(at 203.454 49.276 0)
+		(property "Reference" "LED11"
+			(at 203.962 49.276 0)
 			(effects
 				(font
@@
 			(project "left"
 				(path "/354a5e63-d0f6-4612-b9d9-61a572cb8576"
-					(reference "LED8")
+					(reference "LED11")
 					(unit 1)
 				)
@@
 		(on_board yes)
 		(dnp no)
-		(property "Reference" "LED11"
+		(property "Reference" "LED2"
 			(at 149.606 70.866 0)
 			(effects
@@
 			(project "left"
 				(path "/354a5e63-d0f6-4612-b9d9-61a572cb8576"
-					(reference "LED11")
+					(reference "LED2")
 					(unit 1)
 				)
@@
 		(on_board yes)
 		(dnp no)
-		(property "Reference" "LED16"
+		(property "Reference" "LED1"
 			(at 149.606 92.71 0)
 			(effects
@@
 			(project "left"
 				(path "/354a5e63-d0f6-4612-b9d9-61a572cb8576"
-					(reference "LED16")
+					(reference "LED1")
 					(unit 1)
 				)
@@
 		(on_board yes)
 		(dnp no)
-		(property "Reference" "LED1"
+		(property "Reference" "LED4"
 			(at 148.844 27.686 0)
 			(effects
@@
 			(project "left"
 				(path "/354a5e63-d0f6-4612-b9d9-61a572cb8576"
-					(reference "LED1")
+					(reference "LED4")
 					(unit 1)
 				)
@@
 		(on_board yes)
 		(dnp no)
-		(property "Reference" "LED3"
-			(at 203.708 27.686 0)
+		(property "Reference" "LED12"
+			(at 204.216 27.686 0)
 			(effects
 				(font
@@
 			(project "left"
 				(path "/354a5e63-d0f6-4612-b9d9-61a572cb8576"
-					(reference "LED3")
+					(reference "LED12")
 					(unit 1)
 				)
@@
 		(on_board yes)
 		(dnp no)
-		(property "Reference" "LED17"
+		(property "Reference" "LED5"
 			(at 177.546 92.456 0)
 			(effects
@@
 			(project "left"
 				(path "/354a5e63-d0f6-4612-b9d9-61a572cb8576"
-					(reference "LED17")
+					(reference "LED5")
 					(unit 1)
 				)
@@
 		(on_board yes)
 		(dnp no)
-		(property "Reference" "LED15"
+		(property "Reference" "LED18"
 			(at 257.556 70.866 0)
 			(effects
@@
 			(project "left"
 				(path "/354a5e63-d0f6-4612-b9d9-61a572cb8576"
-					(reference "LED15")
+					(reference "LED18")
 					(unit 1)
 				)
@@
 		(dnp no)
 		(fields_autoplaced yes)
-		(property "Reference" "BT2"
+		(property "Reference" "JST1"
 			(at 146.6215 157.48 90)
 			(effects
@@
 			(project "left"
 				(path "/354a5e63-d0f6-4612-b9d9-61a572cb8576"
-					(reference "BT2")
+					(reference "JST1")
 					(unit 1)
 				)
@@
 		(on_board yes)
 		(dnp no)
-		(property "Reference" "LED6"
+		(property "Reference" "LED3"
 			(at 149.098 49.276 0)
 			(effects
@@
 			(project "left"
 				(path "/354a5e63-d0f6-4612-b9d9-61a572cb8576"
-					(reference "LED6")
+					(reference "LED3")
 					(unit 1)
 				)
@@
 		(on_board yes)
 		(dnp no)
-		(property "Reference" "LED13"
+		(property "Reference" "LED10"
 			(at 204.216 70.866 0)
 			(effects
@@
 			(project "left"
 				(path "/354a5e63-d0f6-4612-b9d9-61a572cb8576"
-					(reference "LED13")
+					(reference "LED10")
 					(unit 1)
 				)
